File: voltage_boost.kicad_pcb (KiCad board)
At the start: 2 copper layers, 99.5 x 62.5 mm, 59 parts, among them J1 Conn_01x02, J2 Conn_01x03, J3 Conn_01x05, J4 Conn_01x02, Q2 IRF9952

Commit message: added readme and screenshots
Parts:
- removed DA5: AD8056, Package_SO:SO-8_3.9x4.9mm_P1.27mm
- removed Q2: IRF9952, Package_SO:SO-8_3.9x4.9mm_P1.27mm
- removed VD10, VD11: BZX55, Diode_THT:D_DO-35_SOD27_P10.16mm_Horizontal
- added DA1: AD8056, Package_SO:SOIC-8_3.9x4.9mm_P1.27mm, F.Cu at (52.0, 49.5)
- added VD1: BZX55, Diode_THT:D_DO-35_SOD27_P10.16mm_Horizontal, B.Cu at (71.7, 35.4)
- added VD2: BZX55, Diode_THT:D_DO-35_SOD27_P10.16mm_Horizontal, B.Cu at (71.9, 39.8)
- added VT2: IRF9952, Package_SO:SOIC-8_3.9x4.9mm_P1.27mm, F.Cu at (47.1, 27.3)
- R61: value 10k -> 1k
Routing:
- net Net-(VD10-Pad1): track 4.73 -> 0.00 mm
- net Net-(VD1-Pad1): track 0.00 -> 4.73 mm
