File: voltage_boost.sch (KiCad schematic (older format))
At the start: 56 parts, among them J1 Conn_01x02, J2 Conn_01x03, J3 Conn_01x05, J4 Conn_01x02, Q2 IRF9952

Commit message: transfered library
Parts:
- removed DA5: AD8056, Package_SO:SO-8_3.9x4.9mm_P1.27mm, symbol Library:AD8056
- removed Q2: IRF9952, Package_SO:SO-8_3.9x4.9mm_P1.27mm, symbol Library:IRF9952
- removed VD10, VD11: BZX55, Diode_THT:D_DO-35_SOD27_P10.16mm_Horizontal, symbol Library:BZX55
- added DA1: AD8056, symbol library:AD8056
- added VD1, VD2: BZX55, symbol library:BZX55
- added VT2: IRF9952, symbol library:IRF9952
Connections:
- net +12V_corr: now also DA1.8
- net -12V_corr: now also DA1.4
- net at R70.1, R75.1, R76.1: now also DA1.3 (+)
- net at R55.1, R62.1, R63.2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: now also DA1.1
- net at C47.1, R54.2, R60.2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: now also DA1.2 (-)
- net at R66.1: now also VT2.4
- net at R63.1: now also VT2.2
- net at C51.2, R79.2, R82.1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: now also VD2.2
- net at R54.1, R73.2, R78.1: now also VT2.1, VT2.3
- net at R65.2: now also VT2.5, VT2.6
- net at R56.2: now also VT2.7, VT2.8
- net at R73.1, R79.1, VT1.1 (G): now also VD1.2
- new net: VD1.1, VD2.1
Changed lines of the file:
@@
 	3350 5410 3350 5310
-$Comp
-L Library:AD8056 DA5
-U 1 1 5FE71019
-P 3950 4810
-F 0 "DA5" H 4100 4960 50  0000 L CNN
-F 1 "AD8056" H 4100 4660 50  0001 L CNN
-F 2 "Package_SO:SO-8_3.9x4.9mm_P1.27mm" H 4180 4990 50  0001 C CNN
-F 3 "" H 4180 4990 50  0001 C CNN
-	1    3950 4810
-	1    0    0    -1
-$EndComp
 $Comp
 L Device:R R60
@@
 	0    1    1    0
 $EndComp
-$Comp
-L Library:IRF9952 Q2
-U 1 1 5FEB2844
-P 5300 4510
-F 0 "Q2" H 5150 4960 50  0000 C CNN
-F 1 "IRF9952" H 5300 4060 50  0000 C CNN
-F 2 "Package_SO:SO-8_3.9x4.9mm_P1.27mm" H 5250 4810 50  0001 C CNN
-F 3 "" H 5250 4810 50  0001 C CNN
-	1    5300 4510
-	1    0    0    -1
-$EndComp
 Wire Wire Line
 	5650 4460 5900 4460
@@
 Wire Wire Line
 	5650 4260 5650 4160
-Connection ~ 5650 4160
 Wire Wire Line
 	5650 4660 5650 4560
-Connection ~ 5650 4560
 $Comp
 L Device:R R56
@@
 Wire Wire Line
 	6900 4860 6550 4860
-Wire Wire Line
-	6900 4860 7400 4860
 Connection ~ 6900 4860
-$Comp
-L Library:BZX55 VD10
-U 1 1 5FECE04E
-P 7400 5010
-F 0 "VD10" V 7446 4932 50  0000 R CNN
-F 1 "BZX55" V 7355 4932 50  0000 R CNN
-F 2 "Diode_THT:D_DO-35_SOD27_P10.16mm_Horizontal" H 7300 5010 50  0001 C CNN
-F 3 "" H 7300 5010 50  0001 C CNN
-	1    7400 5010
-	0    -1   -1   0
-$EndComp
-$Comp
-L Library:BZX55 VD11
-U 1 1 5FED04CB
-P 7400 5310
-F 0 "VD11" V 7354 5397 50  0000 L CNN
-F 1 "BZX55" V 7445 5397 50  0000 L CNN
-F 2 "Diode_THT:D_DO-35_SOD27_P10.16mm_Horizontal" H 7300 5310 50  0001 C CNN
-F 3 "" H 7300 5310 50  0001 C CNN
-	1    7400 5310
-	0    1    1    0
-$EndComp
-Wire Wire Line
-	7400 5460 6900 5460
 Wire Wire Line
 	6900 5010 6900 4860
 Wire Wire Line
 	6900 5460 6900 5310
+$Comp
+L Device:R R82
+U 1 1 5FED74FC
+P 8000 5810
+F 0 "R82" H 8070 5856 50  0000 L CNN
+F 1 "130" H 8070 5765 50  0000 L CNN
+F 2 "Resistor_THT:R_Axial_DIN0617_L17.0mm_D6.0mm_P25.40mm_Horizontal" V 7930 5810 50  0001 C CNN
+F 3 "~" H 8000 5810 50  0001 C CNN
+	1    8000 5810
+	1    0    0    -1
+$EndComp
+Wire Wire Line
+	8000 5060 8000 5460
+Connection ~ 8000 5460
+$Comp
+L Device:R R68
+U 1 1 5FE8F7C3
+P 9400 4560
+F 0 "R68" V 9300 4560 50  0000 C CNN
+F 1 "30" V 9500 4560 50  0000 C CNN
+F 2 "Resistor_THT:R_Axial_DIN0617_L17.0mm_D6.0mm_P25.40mm_Horizontal" V 9330 4560 50  0001 C CNN
+F 3 "~" H 9400 4560 50  0001 C CNN
+	1    9400 4560
+	0    1    1    0
+$EndComp
+Connection ~ 3470 990
+Wire Wire Line
+	3470 990  3820 990
+Connection ~ 4470 990
+Wire Wire Line
+	4120 990  4470 990
+Wire Wire Line
+	3470 990  3370 990
+Wire Wire Line
+	4470 990  4570 990
+Text Label 4570 990  0    50   ~ 0
++12V_corr
+Wire Wire Line
+	4470 1140 4470 990
+$Comp
+L Device:C C41
+U 1 1 5FF238E3
+P 4470 1290
+F 0 "C41" H 4585 1336 50  0000 L CNN
+F 1 "1u" H 4585 1245 50  0000 L CNN
+F 2 "Capacitor_SMD:C_0603_1608Metric" H 4508 1140 50  0001 C CNN
+F 3 "~" H 4470 1290 50  0001 C CNN
+	1    4470 1290
+	1    0    0    -1
+$EndComp
+Wire Wire Line
+	3470 1140 3470 990
+$Comp
+L Device:C C40
+U 1 1 5FF1F0F7
+P 3470 1290
+F 0 "C40" H 3585 1336 50  0000 L CNN
+F 1 "1u" H 3585 1245 50  0000 L CNN
+F 2 "Capacitor_SMD:C_0603_1608Metric" H 3508 1140 50  0001 C CNN
+F 3 "~" H 3470 1290 50  0001 C CNN
+	1    3470 1290
+	1    0    0    -1
+$EndComp
+Wire Wire Line
+	5000 2810 5900 2810
 $Comp
 L Transistor_FET:IRF740 VT1
@@
 	1    0    0    -1
 $EndComp
-Wire Wire Line
-	7700 4860 7400 4860
-Connection ~ 7400 4860
-$Comp
-L Device:R R82
-U 1 1 5FED74FC
-P 8000 5810
-F 0 "R82" H 8070 5856 50  0000 L CNN
-F 1 "130" H 8070 5765 50  0000 L CNN
-F 2 "Resistor_THT:R_Axial_DIN0617_L17.0mm_D6.0mm_P25.40mm_Horizontal" V 7930 5810 50  0001 C CNN
-F 3 "~" H 8000 5810 50  0001 C CNN
-	1    8000 5810
-	1    0    0    -1
-$EndComp
-Wire Wire Line
-	7400 5460 8000 5460
-Connection ~ 7400 5460
-Wire Wire Line
-	8000 5060 8000 5460
-Connection ~ 8000 5460
-$Comp
-L Device:R R68
-U 1 1 5FE8F7C3
-P 9400 4560
-F 0 "R68" V 9300 4560 50  0000 C CNN
-F 1 "30" V 9500 4560 50  0000 C CNN
-F 2 "Resistor_THT:R_Axial_DIN0617_L17.0mm_D6.0mm_P25.40mm_Horizontal" V 9330 4560 50  0001 C CNN
-F 3 "~" H 9400 4560 50  0001 C CNN
-	1    9400 4560
-	0    1    1    0
-$EndComp
-Connection ~ 3470 990
-Wire Wire Line
-	3470 990  3820 990
-Connection ~ 4470 990
-Wire Wire Line
-	4120 990  4470 990
-Wire Wire Line
-	3470 990  3370 990
-Wire Wire Line
-	4470 990  4570 990
-Text Label 4570 990  0    50   ~ 0
-+12V_corr
-Wire Wire Line
-	4470 1140 4470 990
-$Comp
-L Device:C C41
-U 1 1 5FF238E3
-P 4470 1290
-F 0 "C41" H 4585 1336 50  0000 L CNN
-F 1 "1u" H 4585 1245 50  0000 L CNN
-F 2 "Capacitor_SMD:C_0603_1608Metric" H 4508 1140 50  0001 C CNN
-F 3 "~" H 4470 1290 50  0001 C CNN
-	1    4470 1290
-	1    0    0    -1
-$EndComp
-Wire Wire Line
-	3470 1140 3470 990
-$Comp
-L Device:C C40
-U 1 1 5FF1F0F7
-P 3470 1290
-F 0 "C40" H 3585 1336 50  0000 L CNN
-F 1 "1u" H 3585 1245 50  0000 L CNN
-F 2 "Capacitor_SMD:C_0603_1608Metric" H 3508 1140 50  0001 C CNN
-F 3 "~" H 3470 1290 50  0001 C CNN
-	1    3470 1290
-	1    0    0    -1
-$EndComp
-Wire Wire Line
-	5000 2810 5900 2810
+$Comp
+L library:AD8056 DA1
+U 1 1 60463C2E
+P 3950 4810
+F 0 "DA1" H 4150 4670 50  0001 C CNN
+F 1 "AD8056" H 4190 4690 50  0000 L CNN
+F 2 "" H 4280 4940 50  0001 C CNN
+F 3 "" H 4280 4940 50  0001 C CNN
+	1    3950 4810
+	1    0    0    -1
+$EndComp
+$Comp
+L library:IRF9952 VT2
+U 1 1 60464B7C
+P 5300 4510
+F 0 "VT2" H 5325 5085 50  0000 C CNN
+F 1 "IRF9952" H 5325 4994 50  0000 C CNN
+F 2 "" H 5250 4810 50  0001 C CNN
+F 3 "" H 5250 4810 50  0001 C CNN
+	1    5300 4510
+	1    0    0    -1
+$EndComp
+Connection ~ 5650 4560
+Connection ~ 5650 4160
+$Comp
+L library:BZX55 VD1
+U 1 1 60466D21
+P 7470 5010
+F 0 "VD1" V 7516 4932 50  0000 R CNN
+F 1 "BZX55" V 7425 4932 50  0000 R CNN
+F 2 "" H 7370 5010 50  0001 C CNN
+F 3 "" H 7370 5010 50  0001 C CNN
+	1    7470 5010
+	0    -1   -1   0
+$EndComp
+$Comp
+L library:BZX55 VD2
+U 1 1 60467E9F
+P 7470 5310
+F 0 "VD2" V 7424 5397 50  0000 L CNN
+F 1 "BZX55" V 7515 5397 50  0000 L CNN
+F 2 "" H 7370 5310 50  0001 C CNN
+F 3 "" H 7370 5310 50  0001 C CNN
+	1    7470 5310
+	0    1    1    0
+$EndComp
+Wire Wire Line
+	6900 4860 7470 4860
+Connection ~ 7470 4860
+Wire Wire Line
+	7470 4860 7700 4860
+Wire Wire Line
+	6900 5460 7470 5460
+Connection ~ 7470 5460
+Wire Wire Line
+	7470 5460 8000 5460
 Wire Bus Line
 	11000 3930 11000 4830

Commit message: added readme and screenshots
Parts:
- DA1, VT2: footprint (none) -> Package_SO:SOIC-8_3.9x4.9mm_P1.27mm
- VD1, VD2: footprint (none) -> Diode_THT:D_DO-35_SOD27_P10.16mm_Horizontal
Changed lines of the file:
@@
 F 0 "DA1" H 4150 4670 50  0001 C CNN
 F 1 "AD8056" H 4190 4690 50  0000 L CNN
-F 2 "" H 4280 4940 50  0001 C CNN
+F 2 "Package_SO:SOIC-8_3.9x4.9mm_P1.27mm" H 4280 4940 50  0001 C CNN
 F 3 "" H 4280 4940 50  0001 C CNN
 	1    3950 4810
@@
 F 0 "VT2" H 5325 5085 50  0000 C CNN
 F 1 "IRF9952" H 5325 4994 50  0000 C CNN
-F 2 "" H 5250 4810 50  0001 C CNN
+F 2 "Package_SO:SOIC-8_3.9x4.9mm_P1.27mm" H 5250 4810 50  0001 C CNN
 F 3 "" H 5250 4810 50  0001 C CNN
 	1    5300 4510
@@
 F 0 "VD1" V 7516 4932 50  0000 R CNN
 F 1 "BZX55" V 7425 4932 50  0000 R CNN
-F 2 "" H 7370 5010 50  0001 C CNN
+F 2 "Diode_THT:D_DO-35_SOD27_P10.16mm_Horizontal" H 7370 5010 50  0001 C CNN
 F 3 "" H 7370 5010 50  0001 C CNN
 	1    7470 5010
@@
 F 0 "VD2" V 7424 5397 50  0000 L CNN
 F 1 "BZX55" V 7515 5397 50  0000 L CNN
-F 2 "" H 7370 5310 50  0001 C CNN
+F 2 "Diode_THT:D_DO-35_SOD27_P10.16mm_Horizontal" H 7370 5310 50  0001 C CNN
 F 3 "" H 7370 5310 50  0001 C CNN
 	1    7470 5310
